File: CL70_PCB.kicad_pcb (KiCad board)
At the start: 2 copper layers, 343.8 x 98.1 mm, 204 parts, among them J1 AVR-ISP-6, SW1 SW_Push, U1 ATmega32U4-MU, U2 PRTR5V0U2X, Y1 16MHz

Commit message: Add wiring
Parts:
- RC1, RC2: value 22 -> 22k
- RLED1, RLED2, RLED3: value 1k -> 330
- moved SW1 19.4 mm to (361.9, 140.8), turned to 0 degrees
- moved RC3 14.2 mm to (355.4, 139.8), turned to 0 degrees
- moved CRGB12 12.6 mm to (187.2, 176.3)
- moved CRGB5 12.4 mm to (187.0, 119.9)
- moved CRGB8 12.3 mm to (61.5, 120.2)
- moved CRGB7 12.2 mm to (103.5, 119.9)
- moved CRGB11 12.2 mm to (144.8, 177.4)
- moved CRGB6 12.2 mm to (144.8, 119.9)
- moved CRGB10 12.0 mm to (103.2, 177.1)
- moved D71 11.3 mm to (365.8, 163.6)
- moved J1 5.12 mm to (356.7, 163.0)
- moved C2 2.43 mm to (360.7, 149.2)
- moved C3 2.42 mm to (360.6, 146.8)
- moved C8 1.64 mm to (365.6, 171.5)
- moved C9 1.55 mm to (365.6, 169.9)
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Connections:
- RC4 pad 1: Net-(U1-PD0) -> Net-(U1-PD2)
- RC4 pad 2: RESW_A -> RESW_B
- RC5 pad 2: RESW_B -> RESW_A
- S47 pad 1: COL8 -> COL7
- U1 pad 18: Net-(U1-PD0) -> ROW7
- U1 pad 20: ROW9 -> Net-(U1-PD2)
- U1 pad 22: ROW7 -> ROW9
- U1 pad 26: ROW5 -> ROW4
- U1 pad 27: ROW4 -> ROW5
- U1 pad 28: ROW3 -> ROW2
- U1 pad 29: ROW2 -> ROW3
Routing:
- net GND: track 0.00 -> 912.5 mm, vias 0 -> 6
- net +5V: track 0.00 -> 788.1 mm, vias 0 -> 12
- net COL2: track 0.00 -> 469.2 mm, vias 0 -> 1
- net COL1: track 0.00 -> 465.9 mm, vias 0 -> 2
- net COL3: track 0.00 -> 432.2 mm, vias 0 -> 2
- net COL0: track 0.00 -> 420.4 mm, vias 0 -> 1
- net ROW0: track 0.00 -> 399.6 mm, vias 0 -> 4
- net COL4: track 0.00 -> 375.7 mm, vias 0 -> 2
- net ROW3: track 0.00 -> 364.2 mm, vias 0 -> 2
- net ROW1: track 0.00 -> 355.6 mm, vias 0 -> 2
- net ROW8: track 0.00 -> 353.7 mm
- net SLOCK_IND: track 0.00 -> 352.5 mm, vias 0 -> 2
- net CAPS_IND: track 0.00 -> 349.7 mm, vias 0 -> 2
- net LAYER_IND: track 0.00 -> 342.4 mm, vias 0 -> 2
- net ROW2: track 0.00 -> 340.6 mm
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